Commit message: [simulation] Fix contact equation by replacing freeflyer by linear + angular joints
Previous simulation was simulating a spherical contact, not a cylinder.
This made the simulation work in the sagittal plane only.
This is fixed here by removing the freeflyer, and using instead
XY translation joints + rpy angles.

File: simulation/urdf/claptrap.urdf (robot description, URDF)
Before this commit: robot Claptrap, 4 links, 3 joints
Links:
- removed link WheelRim
- added link AnchorRollLink
- added link AnchorXLink
- added link AnchorYLink
- added link AnchorYawLink
- link Body: mass 10.0 -> 3.0
- link Wheel: mass 3.0 -> 1.0
Joints:
- removed joint RimJoint
- added joint AnchorRollJoint: type revolute, parent AnchorYawLink, child AnchorRollLink, origin xyz=0.0 0.0 0.0 rpy=0.0 0.0 0.0, axis 1 0 0, limit effort=1000.0 velocity=1000.0
- added joint AnchorXJoint: type prismatic, parent world, child AnchorXLink, origin xyz=0.0 0.0 0.0 rpy=0.0 0.0 0.0, axis 1 0 0, limit effort=1000.0 velocity=1000.0
- added joint AnchorYJoint: type prismatic, parent AnchorXLink, child AnchorYLink, origin xyz=0.0 0.0 0.0 rpy=0.0 0.0 0.0, axis 0 1 0, limit effort=1000.0 velocity=1000.0
- added joint AnchorYawJoint: type revolute, parent AnchorYLink, child AnchorYawLink, origin xyz=0.0 0.0 0.0 rpy=0.0 0.0 0.0, axis 0 0 1, limit effort=1000.0 velocity=1000.0
- joint BodyJoint: axis (none) -> 0 1 0; origin xyz=0.0 0.0 0.0 rpy=0.0 0.0 0.0 -> xyz=0.0 0.0 0.15 rpy=0.0 0.0 0.0; parent world -> AnchorRollLink; type fixed -> revolute
